File: hardware/lcd-128x64.kicad_pcb (KiCad board)
At the start: 2 copper layers, 85 x 55 mm, 41 parts, among them P1 CON-SENSOR2, P2 Debug, P3 BOOT, P4 CON_4Wire_ER-TP028-1, Q1 2N7002, U1 XMC130024, U2 TSC2046E, U3 LCD-ERC12864, U4 DRILL, U5 DRILL, U6 DRILL, U7 DRILL

Commit message: specify resistor according to production
Parts:
- R9: value 27|22 -> 27
Changed lines of the file:
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@@
       (effects (font (size 0.3 0.3) (thickness 0.075)))
     )
-    (fp_text value 27|22 (at 0 -0.65 180) (layer F.Fab)
+    (fp_text value 27 (at 0 -0.65 180) (layer F.Fab)
       (effects (font (size 0.3 0.3) (thickness 0.075)))
     )
